File: oled_keyboard/oled_keyboard.kicad_sch (KiCad schematic)
At the start: 126 parts, among them J1 Conn_01x20_Socket, J10 Conn_01x20_Socket, J11 Conn_01x20_Socket, J12 Conn_01x20_Socket, J2 Conn_01x20_Socket, J3 Conn_01x20_Socket, J4 Conn_01x20_Socket, J5 Conn_01x20_Socket, J6 Conn_01x20_Socket, J7 Conn_01x20_Socket, J8 Conn_01x20_Socket, J9 Conn_01x20_Socket, SW1 SW_Push, SW10 SW_Push, SW11 SW_Push, SW12 SW_Push, SW2 SW_Push, SW3 SW_Push, SW4 SW_Push, SW5 SW_Push, SW6 SW_Push, SW7 SW_Push, SW8 SW_Push, SW9 SW_Push, U1 TPS61088RHLR

Commit message: fix: added 3v3! enlarged holes for passing naps
Parts:
- added TP9: TestPoint, TestPoint:TestPoint_Pad_D2.5mm, symbol Connector:TestPoint
Connections:
- net MOSI: no longer TP4.1
- net SCK: no longer TP5.1
- net SCLK: now also TP5.1
- net SDIN: now also TP4.1
- net 3V3: now reaches C52.1, C56.1, J9.3 (Pin_3)
- net 3V3: now also A1.36 (3V3), C18.1, C19.1, C2.1, C21.1, C23.1, C24.1, C26.1, C31.1, C35.1, C36.1, C37.1, C38.1, C4.1, C40.1, C41.1, C42.1, C47.1, C51.1, C53.1, C54.1, C57.1, C58.1, J1.3 (Pin_3), J10.3 (Pin_3), J11.3 (Pin_3), J12.3 (Pin_3), J2.3 (Pin_3), J3.3 (Pin_3), J4.3 (Pin_3), J5.3 (Pin_3), J6.3 (Pin_3), J7.3 (Pin_3), J8.3 (Pin_3), TP9.1
