File: oled_keyboard/oled_keyboard.kicad_sch (KiCad schematic)
At the start: 127 parts, among them J1 Conn_01x20_Socket, J10 Conn_01x20_Socket, J11 Conn_01x20_Socket, J12 Conn_01x20_Socket, J2 Conn_01x20_Socket, J3 Conn_01x20_Socket, J4 Conn_01x20_Socket, J5 Conn_01x20_Socket, J6 Conn_01x20_Socket, J7 Conn_01x20_Socket, J8 Conn_01x20_Socket, J9 Conn_01x20_Socket, SW1 SW_Push, SW10 SW_Push, SW11 SW_Push, SW12 SW_Push, SW2 SW_Push, SW3 SW_Push, SW4 SW_Push, SW5 SW_Push, SW6 SW_Push, SW7 SW_Push, SW8 SW_Push, SW9 SW_Push, U1 TPS61088RHLR

Commit message: feat: changed fpc connectors
Parts:
- added H1, H2, H3, H4: MountingHole, MountingHole:MountingHole_2.7mm_M2.5, symbol Mechanical:MountingHole
- J1, J10, J11, J12, J2, J3, J4, J5, J6, J7, J8, J9: footprint 20pin_connector:HRS_TF31-20S-0.5SH_800_ -> 20pin_conn_vert:TE_2-1734742-0
Connections:
- net COL1: now also A1.4 (GPIO2); no longer A1.5 (GPIO3)
- net ROW1: now also A1.5 (GPIO3); no longer A1.4 (GPIO2)
