File: oled_keyboard/oled_keyboard.kicad_sch (KiCad schematic)
At the start: 131 parts, among them J1 Conn_01x20_Socket, J10 Conn_01x20_Socket, J11 Conn_01x20_Socket, J12 Conn_01x20_Socket, J2 Conn_01x20_Socket, J3 Conn_01x20_Socket, J4 Conn_01x20_Socket, J5 Conn_01x20_Socket, J6 Conn_01x20_Socket, J7 Conn_01x20_Socket, J8 Conn_01x20_Socket, J9 Conn_01x20_Socket, SW1 SW_Push, SW10 SW_Push, SW11 SW_Push, SW12 SW_Push, SW2 SW_Push, SW3 SW_Push, SW4 SW_Push, SW5 SW_Push, SW6 SW_Push, SW7 SW_Push, SW8 SW_Push, SW9 SW_Push, U1 TPS61088RHLR

Commit message: release v4.0
Connections:
- net GND: no longer A1.37 (3V3_EN)
Changed lines of the file:
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@@
 	(wire
 		(pts
-			(xy 440.69 149.86) (xy 447.04 149.86)
-		)
-		(stroke
-			(width 0)
-			(type default)
-		)
-	)
-	(wire
-		(pts
 			(xy 304.8 222.25) (xy 304.8 220.98)
 		)
@@
 					(unit 1)
 				)
-			)
-		)
-	)
-	(symbol
-		(lib_id "power:GND")
-		(at 440.69 149.86 270)
-		(unit 1)
-		(exclude_from_sim no)
-		(in_bom yes)
-		(on_board yes)
-		(dnp no)
-		(fields_autoplaced yes)
-		(property "Reference" "#PWR063"
-			(at 434.34 149.86 0)
-			(effects
-				(font
-					(size 1.27 1.27)
-				)
-				(hide yes)
-			)
-		)
-		(property "Value" "GND"
-			(at 436.88 149.8599 90)
-			(effects
-				(font
-					(size 1.27 1.27)
-				)
-				(justify right)
-			)
-		)
-		(property "Footprint" ""
-			(at 440.69 149.86 0)
-			(effects
-				(font
-					(size 1.27 1.27)
-				)
-				(hide yes)
-			)
-		)
-		(property "Datasheet" ""
-			(at 440.69 149.86 0)
-			(effects
-				(font
-					(size 1.27 1.27)
-				)
-				(hide yes)
-			)
-		)
-		(property "Description" "Power symbol creates a global label with name \"GND\" , ground"
-			(at 440.69 149.86 0)
-			(effects
-				(font
-					(size 1.27 1.27)
-				)
-				(hide yes)
-			)
-		)
-		(pin "1"
-		)
-		(instances
-			(project "oled_keyboard"
-				(path "/93cb1d80-50e0-4756-95e4-c1195d62fad8"
-					(reference "#PWR063")
-					(unit 1)
-				)

Commit message: release v5.2
Parts:
- removed TP4, TP5: TestPoint, TestPoint:TestPoint_Pad_D2.5mm, symbol Connector:TestPoint
- added C60, C61, C62, C63, C64, C65, C66, C67, C68, C69, C70, C71: 0.1uF, Capacitor_SMD:C_0603_1608Metric, symbol Device:C
- added R20, R21, R22, R23, R24, R25, R26, R27, R28, R29, R30, R31: 10K, Resistor_SMD:R_0603_1608Metric, symbol Device:R
Connections:
- net 3V3: now also R20.1, R21.1, R22.1, R23.1, R24.1, R25.1, R26.1, R27.1, R28.1, R29.1, R30.1, R31.1
- net CS1: now also R20.2
- net CS10: now also R29.2
- net CS11: now also R30.2
- net CS12: now also R31.2
- net CS2: now also R21.2
- net CS3: now also R22.2
- net CS4: now also R23.2
- net CS5: now also R24.2
- net CS6: now also R25.2
- net CS7: now also R26.2
- net CS8: now also R27.2
- net CS9: now also R28.2
- net DC: now also A1.32 (GPIO27_ADC1); no longer A1.31 (GPIO26_ADC0)
- net GND: now also J1.1 (Pin_1), J1.2 (Pin_2), J1.20 (Pin_20), J10.1 (Pin_1), J10.2 (Pin_2), J10.20 (Pin_20), J11.1 (Pin_1), J11.2 (Pin_2), J11.20 (Pin_20), J12.1 (Pin_1), J12.2 (Pin_2), J12.20 (Pin_20), J2.1 (Pin_1), J2.2 (Pin_2), J2.20 (Pin_20), J3.1 (Pin_1), J3.2 (Pin_2), J3.20 (Pin_20), J4.1 (Pin_1), J4.2 (Pin_2), J4.20 (Pin_20), J5.1 (Pin_1), J5.2 (Pin_2), J5.20 (Pin_20), J6.1 (Pin_1), J6.2 (Pin_2), J6.20 (Pin_20), J7.1 (Pin_1), J7.2 (Pin_2), J7.20 (Pin_20), J8.1 (Pin_1), J8.2 (Pin_2), J8.20 (Pin_20), J9.1 (Pin_1), J9.2 (Pin_2), J9.20 (Pin_20), C60.2, C61.2, C62.2, C63.2, C64.2, C65.2, C66.2, C67.2, C68.2, C69.2, C70.2, C71.2
- net MOSI: now also R19.1; no longer R19.2
- net RES: now also A1.31 (GPIO26_ADC0); no longer A1.32 (GPIO27_ADC1)
- net SCK: now also R18.1; no longer R18.2
- net SCLK: now also R18.2; no longer R18.1
- net SDIN: now also R19.2; no longer R19.1
- net at C48.1, J9.18 (Pin_18): now also C71.1
- net at C34.1, J7.18 (Pin_18): now also C66.1
- net at C25.1, J4.18 (Pin_18): now also C63.1
- net at C17.1, J2.18 (Pin_18): now also C61.1
- net at C49.1, J10.18 (Pin_18): now also C70.1
- net at C22.1, J3.18 (Pin_18): now also C62.1
- net at C32.1, J5.18 (Pin_18): now also C64.1
- net at C50.1, J11.18 (Pin_18): now also C69.1
- net at C39.1, J8.18 (Pin_18): now also C67.1
- net at C1.1, J1.18 (Pin_18): now also C60.1
- net at C55.1, J12.18 (Pin_18): now also C68.1
- net at C33.1, J6.18 (Pin_18): now also C65.1
- no-connect marks 135 -> 99
Other:
- note added: "buffer"
- moved on the sheet: A1, D1, D10, D11, D12, D2, D3, D4, D5, D6, D7, D8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
