File: oled_keyboard/oled_keyboard.kicad_pcb (KiCad board)
At the start: 4 copper layers, 100 x 100 mm, 127 parts, among them J1 Conn_01x20_Socket, J10 Conn_01x20_Socket, J11 Conn_01x20_Socket, J12 Conn_01x20_Socket, J2 Conn_01x20_Socket, J3 Conn_01x20_Socket, J4 Conn_01x20_Socket, J5 Conn_01x20_Socket, J6 Conn_01x20_Socket, J7 Conn_01x20_Socket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

Commit message: released v3.1
Routing:
- net 3V3: track 360.2 -> 361.9 mm
- net VCC: track 406.1 -> 407.9 mm
Other:
- board text added: "oled keyboard v3.1 by Xin 2026.6.23"
- board text removed: "oled keyboard v3.0 by Xin 2026.5.26"
Changed lines of the file:
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@@
 		(layer "F.Fab")
 	)
-	(gr_text "oled keyboard \nv3.0\nby Xin \n2026.5.26"
+	(gr_text "oled keyboard \nv3.1\nby Xin \n2026.6.23"
 		(at 103.124 86.614 90)
 		(layer "B.SilkS")
@@
 	)
 	(segment
+		(start 149.7 54)
+		(end 168.9 54)
+		(width 0.4)
+		(layer "F.Cu")
+		(net 4)
+	)
+	(segment
 		(start 151.725 116.4)
 		(end 168.225 116.4)
@@
 	)
 	(segment
-		(start 168.25 54)
-		(end 168.75 54)
-		(width 0.4)
-		(layer "F.Cu")
-		(net 4)
-	)
-	(segment
-		(start 130.5 54)
-		(end 135 54)
-		(width 0.4)
-		(layer "F.Cu")
-		(net 4)
-	)
-	(segment
 		(start 173.5 74.75)
 		(end 173.75 74.5)
@@
 	)
 	(segment
-		(start 135 54)
-		(end 135.324 54)
-		(width 0.4)
-		(layer "F.Cu")
-		(net 4)
-	)
-	(segment
 		(start 130.475 116.4)
 		(end 134.975 116.4)
@@
 	)
 	(segment
-		(start 135 54)
-		(end 151.75 54)
+		(start 130.5 54)
+		(end 149.7 54)
 		(width 0.4)
 		(layer "F.Cu")
@@
 	)
 	(segment
-		(start 151.75 54)
-		(end 152 54)
-		(width 0.4)
-		(layer "F.Cu")
-		(net 4)
-	)
-	(segment
 		(start 168.225 116.4)
 		(end 168.725 116.4)
@@
 	)
 	(segment
-		(start 151.75 54)
-		(end 168.25 54)
-		(width 0.4)
-		(layer "F.Cu")
-		(net 4)
-	)
-	(segment
 		(start 168.25 54)
 		(end 173.75 54)
@@
 	)
 	(segment
+		(start 105.39 42.5675)
+		(end 124.3175 42.5675)
+		(width 0.4)
+		(layer "B.Cu")
+		(net 4)
+	)
+	(segment
 		(start 127.568705 115.206295)
 		(end 126.775 116)
@@
 	)
 	(segment
+		(start 129.75 49)
+		(end 130.448223 49.698223)
+		(width 0.4)
+		(layer "B.Cu")
+		(net 4)
+	)
+	(segment
 		(start 168.823223 95.548223)
 		(end 168.823223 94.406295)
@@
 	)
 	(segment
-		(start 116.5 47)
-		(end 125 47)
+		(start 125.25 47.25)
+		(end 127 49)
 		(width 0.4)
 		(layer "B.Cu")
@@
 	)
 	(segment
+		(start 124.3175 42.5675)
+		(end 125.25 43.5)
+		(width 0.4)
+		(layer "B.Cu")
+		(net 4)
+	)
+	(segment
 		(start 127.593705 52.806295)
 		(end 126.8 53.6)
@@
 	)
 	(segment
-		(start 112.0675 42.5675)
-		(end 116.5 47)
-		(width 0.4)
-		(layer "B.Cu")
-		(net 4)
-	)
-	(segment
 		(start 168.875 116.4)
 		(end 168.823223 116.348223)
@@
 	)
 	(segment
-		(start 125 47)
-		(end 127 49)
-		(width 0.4)
-		(layer "B.Cu")
-		(net 4)
-	)
-	(segment
 		(start 149.675 95.6)
 		(end 149.623223 95.548223)
@@
 	)
 	(segment
+		(start 125.25 43.5)
+		(end 125.25 47.25)
+		(width 0.4)
+		(layer "B.Cu")
+		(net 4)
+	)
+	(segment
 		(start 171.989341 116.4)
 		(end 173.75 114.639341)
@@
 	)
 	(segment
-		(start 129.75 49)
-		(end 130.448223 49.698223)
-		(width 0.4)
-		(layer "B.Cu")
-		(net 4)
-	)
-	(segment
 		(start 145.975 116)
 		(end 145.975 117)
@@
 	)
 	(segment
-		(start 127 49)
-		(end 129.75 49)
-		(width 0.4)
-		(layer "B.Cu")
-		(net 4)
-	)
-	(segment
 		(start 126.775 74.4)
 		(end 126.775 75.4)
@@
 	)
 	(segment
+		(start 127 49)
+		(end 129.75 49)
+		(width 0.4)
+		(layer "B.Cu")
+		(net 4)
+	)
+	(segment
 		(start 173.75 114.639341)
 		(end 173.75 74.5)
@@
 	)
 	(segment
-		(start 130.448223 49.698223)
-		(end 130.448223 51.2)
-		(width 0.4)
-		(layer "B.Cu")
-		(net 4)
-	)
-	(segment
 		(start 168.848223 52.806295)
 		(end 165.993705 52.806295)
@@
 	)
 	(segment
-		(start 105.39 42.5675)
-		(end 112.0675 42.5675)
+		(start 130.448223 49.698223)
+		(end 130.448223 51.2)
 		(width 0.4)
 		(layer "B.Cu")
@@
 	)
 	(segment
+		(start 116 117.15)
+		(end 115.5 116.65)
+		(width 0.5)
+		(layer "F.Cu")
+		(net 43)
+	)
+	(segment
 		(start 106.8 127.75)
 		(end 103.8555 127.75)
@@
 	)
 	(segment
+		(start 117.275 117.15)
+		(end 116 117.15)
+		(width 0.5)
+		(layer "F.Cu")
+		(net 43)
+	)
+	(segment
 		(start 94.7755 103.562)
 		(end 94.7755 104.319)
@@
 		(layer "F.Cu")
 		(net 43)
-	)
-	(segment
-		(start 153.5 54.75)
-		(end 153.75 54.75)
-		(width 0.5)
-		(layer "F.Cu")
-		(net 43)
